Commit message: Added working quadruped gazebo simulation

File: ROS/catkin_ws_quad/quadruped_description/urdf/quadruped.xacro (robot description, xacro)
@@ -6,7 +6,7 @@
 <link name="base_link">
   <inertial>
-    <origin rpy="0 0 0" xyz="-4.417326064147873e-17 1.940982339223468e-16 0.04901709635318994"/>
-    <mass value="201.8775331511704"/>
-    <inertia ixx="7.191605" ixy="-1.1e-05" ixz="-0.0" iyy="2.82248" iyz="0.0" izz="9.659005"/>
+    <origin rpy="0 0 0" xyz="-3.431576713324414e-17 2.610567498014317e-16 0.04324730691236673"/>
+    <mass value="29.384744866709624"/>
+    <inertia ixx="1.089951" ixy="-1.1e-05" ixz="0.0" iyy="0.445316" iyz="0.0" izz="1.461435"/>
   </inertial>
   <visual>
@@ -66,5 +66,5 @@
 <link name="link1FrontLeft_1">
   <inertial>
-    <origin rpy="0 0 0" xyz="-0.006632742807460124 -0.00889229477475234 -0.06827854152055422"/>
+    <origin rpy="0 0 0" xyz="-0.006632742807460124 -0.008892294774752285 -0.06827854152055422"/>
     <mass value="0.6959462012084651"/>
     <inertia ixx="0.00104" ixy="-4.6e-05" ixz="-5.5e-05" iyy="0.000651" iyz="-0.000304" izz="0.000853"/>
@@ -106,7 +106,7 @@
 <link name="link2FrontRight_1">
   <inertial>
-    <origin rpy="0 0 0" xyz="0.04835689837404811 3.830943160643141e-06 -0.20537104153229047"/>
+    <origin rpy="0 0 0" xyz="0.04835689837404797 0.1778581520813298 -0.1026823777545005"/>
     <mass value="0.8659841478355499"/>
-    <inertia ixx="0.00672" ixy="-0.0" ixz="0.000112" iyy="0.007032" iyz="-1e-05" izz="0.000496"/>
+    <inertia ixx="0.00672" ixy="-9.7e-05" ixz="5.5e-05" iyy="0.002139" iyz="0.002835" izz="0.005389"/>
   </inertial>
   <visual>
@@ -126,7 +126,7 @@
 <link name="link2BackLeft_1">
   <inertial>
-    <origin rpy="0 0 0" xyz="-0.04835689837407542 -3.830943160643141e-06 -0.20537104153228802"/>
+    <origin rpy="0 0 0" xyz="-0.04835689837407095 -0.20225131512422015 -0.035658823063442355"/>
     <mass value="0.8659841478355499"/>
-    <inertia ixx="0.00672" ixy="-0.0" ixz="-0.000112" iyy="0.007032" iyz="1e-05" izz="0.000496"/>
+    <inertia ixx="0.00672" ixy="-0.00011" ixz="-1.9e-05" iyy="0.000697" iyz="-0.001127" izz="0.006832"/>
   </inertial>
   <visual>
@@ -146,7 +146,7 @@
 <link name="link2FrontLeft_1">
   <inertial>
-    <origin rpy="0 0 0" xyz="-0.04835589963015452 -3.830943160254563e-06 -0.20537104153228863"/>
+    <origin rpy="0 0 0" xyz="-0.048355899630154325 0.17785432113816846 -0.10268901314269395"/>
     <mass value="0.8659841478355499"/>
-    <inertia ixx="0.00672" ixy="-0.0" ixz="-0.000112" iyy="0.007032" iyz="-1.1e-05" izz="0.000496"/>
+    <inertia ixx="0.00672" ixy="9.7e-05" ixz="-5.6e-05" iyy="0.00214" iyz="0.002836" izz="0.005388"/>
   </inertial>
   <visual>
@@ -166,7 +166,7 @@
 <link name="link2BackRight_1">
   <inertial>
-    <origin rpy="0 0 0" xyz="0.04835589963013884 3.830943160532119e-06 -0.2053710415322919"/>
+    <origin rpy="0 0 0" xyz="0.04835589963013057 -0.20224998465162836 -0.03566636854848647"/>
     <mass value="0.8659841478355499"/>
-    <inertia ixx="0.00672" ixy="-0.0" ixz="0.000112" iyy="0.007032" iyz="1.1e-05" izz="0.000496"/>
+    <inertia ixx="0.00672" ixy="0.00011" ixz="2e-05" iyy="0.000697" iyz="-0.001129" izz="0.006831"/>
   </inertial>
   <visual>
@@ -186,10 +186,10 @@
 <link name="link3FrontRight_1">
   <inertial>
-    <origin rpy="0 0 0" xyz="0.04813339309281514 2.7563511140193953e-06 -0.22442742342969874"/>
+    <origin rpy="0 0 0" xyz="0.04813339309281217 -0.14425715774798153 -0.1719240538952389"/>
     <mass value="0.8975642770404472"/>
-    <inertia ixx="0.00868" ixy="-0.0" ixz="0.000137" iyy="0.008993" iyz="1.4e-05" izz="0.000506"/>
-  </inertial>
-  <visual>
-    <origin rpy="0 0 0" xyz="0.196988 0.290812 0.357157"/>
+    <inertia ixx="0.00868" ixy="8.8e-05" ixz="0.000106" iyy="0.005501" iyz="-0.004176" izz="0.003999"/>
+  </inertial>
+  <visual>
+    <origin rpy="0 0 0" xyz="0.196988 0.068949 0.229078"/>
     <geometry>
       <mesh filename="package://quadruped_description/meshes/link3FrontRight_1.stl" scale="0.001 0.001 0.001"/>
@@ -198,5 +198,5 @@
   </visual>
   <collision>
-    <origin rpy="0 0 0" xyz="0.196988 0.290812 0.357157"/>
+    <origin rpy="0 0 0" xyz="0.196988 0.068949 0.229078"/>
     <geometry>
       <mesh filename="package://quadruped_description/meshes/link3FrontRight_1.stl" scale="0.001 0.001 0.001"/>
@@ -206,10 +206,10 @@
 <link name="link3BackLeft__1">
   <inertial>
-    <origin rpy="0 0 0" xyz="-0.04813239309295386 -2.7563511141304176e-06 -0.2244274234296863"/>
+    <origin rpy="0 0 0" xyz="-0.04813239309292175 0.1442566121913428 -0.17192326751708192"/>
     <mass value="0.8975642770404472"/>
-    <inertia ixx="0.00868" ixy="-0.0" ixz="-0.000137" iyy="0.008993" iyz="-1.4e-05" izz="0.000506"/>
-  </inertial>
-  <visual>
-    <origin rpy="0 0 0" xyz="-0.196987 -0.290812 0.357157"/>
+    <inertia ixx="0.00868" ixy="8.8e-05" ixz="-0.000106" iyy="0.005501" iyz="0.004176" izz="0.003999"/>
+  </inertial>
+  <visual>
+    <origin rpy="0 0 0" xyz="-0.196987 -0.038516 0.145476"/>
     <geometry>
       <mesh filename="package://quadruped_description/meshes/link3BackLeft__1.stl" scale="0.001 0.001 0.001"/>
@@ -218,5 +218,5 @@
   </visual>
   <collision>
-    <origin rpy="0 0 0" xyz="-0.196987 -0.290812 0.357157"/>
+    <origin rpy="0 0 0" xyz="-0.196987 -0.038516 0.145476"/>
     <geometry>
       <mesh filename="package://quadruped_description/meshes/link3BackLeft__1.stl" scale="0.001 0.001 0.001"/>
@@ -226,10 +226,10 @@
 <link name="link3FrontLeft_1">
   <inertial>
-    <origin rpy="0 0 0" xyz="-0.04813211460166608 -3.756351113770595e-06 -0.22442742342969108"/>
+    <origin rpy="0 0 0" xyz="-0.04813211460165709 -0.14426164676732856 -0.1719192169758414"/>
     <mass value="0.8975642770404472"/>
-    <inertia ixx="0.00868" ixy="-0.0" ixz="-0.000137" iyy="0.008993" iyz="1.3e-05" izz="0.000506"/>
-  </inertial>
-  <visual>
-    <origin rpy="0 0 0" xyz="-0.197012 0.290787 0.357157"/>
+    <inertia ixx="0.00868" ixy="-8.9e-05" ixz="-0.000105" iyy="0.005499" iyz="-0.004177" izz="0.004"/>
+  </inertial>
+  <visual>
+    <origin rpy="0 0 0" xyz="-0.197012 0.068937 0.229057"/>
     <geometry>
       <mesh filename="package://quadruped_description/meshes/link3FrontLeft_1.stl" scale="0.001 0.001 0.001"/>
@@ -238,5 +238,5 @@
   </visual>
   <collision>
-    <origin rpy="0 0 0" xyz="-0.197012 0.290787 0.357157"/>
+    <origin rpy="0 0 0" xyz="-0.197012 0.068937 0.229057"/>
     <geometry>
       <mesh filename="package://quadruped_description/meshes/link3FrontLeft_1.stl" scale="0.001 0.001 0.001"/>
@@ -246,10 +246,10 @@
 <link name="link3BackRight_1">
   <inertial>
-    <origin rpy="0 0 0" xyz="0.04813311460158362 2.7563511140193953e-06 -0.2244274234297003"/>
+    <origin rpy="0 0 0" xyz="0.04813311460159092 0.14426226000625303 -0.1719194610389605"/>
     <mass value="0.8975642770404472"/>
-    <inertia ixx="0.00868" ixy="-0.0" ixz="0.000137" iyy="0.008993" iyz="-1.3e-05" izz="0.000506"/>
-  </inertial>
-  <visual>
-    <origin rpy="0 0 0" xyz="0.197013 -0.290788 0.357157"/>
+    <inertia ixx="0.00868" ixy="-8.9e-05" ixz="0.000105" iyy="0.005499" iyz="0.004177" izz="0.004"/>
+  </inertial>
+  <visual>
+    <origin rpy="0 0 0" xyz="0.197013 -0.038511 0.145451"/>
     <geometry>
       <mesh filename="package://quadruped_description/meshes/link3BackRight_1.stl" scale="0.001 0.001 0.001"/>
@@ -258,5 +258,5 @@
   </visual>
   <collision>
-    <origin rpy="0 0 0" xyz="0.197013 -0.290788 0.357157"/>
+    <origin rpy="0 0 0" xyz="0.197013 -0.038511 0.145451"/>
     <geometry>
       <mesh filename="package://quadruped_description/meshes/link3BackRight_1.stl" scale="0.001 0.001 0.001"/>
@@ -266,10 +266,10 @@
 <link name="link4FrontRight_1">
   <inertial>
-    <origin rpy="0 0 0" xyz="0.04421036643334067 -0.006254524034631337 -0.10914906216532516"/>
+    <origin rpy="0 0 0" xyz="0.04421036643333587 -0.0949469816012059 -0.054201739043747255"/>
     <mass value="0.3651188269789837"/>
-    <inertia ixx="0.001791" ixy="-5e-06" ixz="-7.1e-05" iyy="0.0019" iyz="-0.000199" izz="0.000283"/>
-  </inertial>
-  <visual>
-    <origin rpy="0 0 0" xyz="0.196988 0.290825 0.641575"/>
+    <inertia ixx="0.001791" ixy="-6.3e-05" ixz="-3.4e-05" iyy="0.000581" iyz="-0.000658" izz="0.001602"/>
+  </inertial>
+  <visual>
+    <origin rpy="0 0 0" xyz="0.196988 0.251779 0.446947"/>
     <geometry>
       <mesh filename="package://quadruped_description/meshes/link4FrontRight_1.stl" scale="0.001 0.001 0.001"/>
@@ -278,5 +278,5 @@
   </visual>
   <collision>
-    <origin rpy="0 0 0" xyz="0.196988 0.290825 0.641575"/>
+    <origin rpy="0 0 0" xyz="0.196988 0.251779 0.446947"/>
     <geometry>
       <mesh filename="package://quadruped_description/meshes/link4FrontRight_1.stl" scale="0.001 0.001 0.001"/>
@@ -286,10 +286,10 @@
 <link name="link4BackLeft_1">
   <inertial>
-    <origin rpy="0 0 0" xyz="-0.044409351302915484 -0.0062299379155703605 -0.10914906216527487"/>
+    <origin rpy="0 0 0" xyz="-0.04440935130285234 -0.05996987904558257 -0.09141047421903997"/>
     <mass value="0.3651188269789837"/>
-    <inertia ixx="0.001791" ixy="5e-06" ixz="7.1e-05" iyy="0.0019" iyz="-0.000199" izz="0.000283"/>
-  </inertial>
-  <visual>
-    <origin rpy="0 0 0" xyz="-0.196987 -0.290825 0.641575"/>
+    <inertia ixx="0.001791" ixy="4.1e-05" ixz="5.9e-05" iyy="0.001323" iyz="-0.0008" izz="0.00086"/>
+  </inertial>
+  <visual>
+    <origin rpy="0 0 0" xyz="-0.196987 -0.221346 0.363345"/>
     <geometry>
       <mesh filename="package://quadruped_description/meshes/link4BackLeft_1.stl" scale="0.001 0.001 0.001"/>
@@ -298,5 +298,5 @@
   </visual>
   <collision>
-    <origin rpy="0 0 0" xyz="-0.196987 -0.290825 0.641575"/>
+    <origin rpy="0 0 0" xyz="-0.196987 -0.221346 0.363345"/>
     <geometry>
       <mesh filename="package://quadruped_description/meshes/link4BackLeft_1.stl" scale="0.001 0.001 0.001"/>
@@ -306,10 +306,10 @@
 <link name="link4FrontLeft_1">
   <inertial>
-    <origin rpy="0 0 0" xyz="-0.0444093513027308 -0.006229937915569972 -0.10914906216529474"/>
+    <origin rpy="0 0 0" xyz="-0.04440935130271231 -0.0949329399299435 -0.054221777753314326"/>
     <mass value="0.3651188269789837"/>
-    <inertia ixx="0.001791" ixy="5e-06" ixz="7.1e-05" iyy="0.0019" iyz="-0.000199" izz="0.000283"/>
-  </inertial>
-  <visual>
-    <origin rpy="0 0 0" xyz="-0.197012 0.290775 0.641575"/>
+    <inertia ixx="0.001791" ixy="6.3e-05" ixz="3.4e-05" iyy="0.000581" iyz="-0.000658" izz="0.001602"/>
+  </inertial>
+  <visual>
+    <origin rpy="0 0 0" xyz="-0.197012 0.251748 0.446942"/>
     <geometry>
       <mesh filename="package://quadruped_description/meshes/link4FrontLeft_1.stl" scale="0.001 0.001 0.001"/>
@@ -318,5 +318,5 @@
   </visual>
   <collision>
-    <origin rpy="0 0 0" xyz="-0.197012 0.290775 0.641575"/>
+    <origin rpy="0 0 0" xyz="-0.197012 0.251748 0.446942"/>
     <geometry>
       <mesh filename="package://quadruped_description/meshes/link4FrontLeft_1.stl" scale="0.001 0.001 0.001"/>
@@ -326,10 +326,10 @@
 <link name="link4FrontRight__1__1">
   <inertial>
-    <origin rpy="0 0 0" xyz="0.04441036643333646 -0.006254524034631559 -0.10914906216532572"/>
+    <origin rpy="0 0 0" xyz="0.04440936643334964 -0.05999066356480873 -0.09139863065595971"/>
     <mass value="0.3651188269789837"/>
-    <inertia ixx="0.001791" ixy="-5e-06" ixz="-7.1e-05" iyy="0.0019" iyz="-0.000199" izz="0.000283"/>
-  </inertial>
-  <visual>
-    <origin rpy="0 0 0" xyz="0.197013 -0.290775 0.641575"/>
+    <inertia ixx="0.001791" ixy="-4e-05" ixz="-5.9e-05" iyy="0.001323" iyz="-0.0008" izz="0.00086"/>
+  </inertial>
+  <visual>
+    <origin rpy="0 0 0" xyz="0.197012 -0.221322 0.363336"/>
     <geometry>
       <mesh filename="package://quadruped_description/meshes/link4FrontRight__1__1.stl" scale="0.001 0.001 0.001"/>
@@ -338,5 +338,5 @@
   </visual>
   <collision>
-    <origin rpy="0 0 0" xyz="0.197013 -0.290775 0.641575"/>
+    <origin rpy="0 0 0" xyz="0.197012 -0.221322 0.363336"/>
     <geometry>
       <mesh filename="package://quadruped_description/meshes/link4FrontRight__1__1.stl" scale="0.001 0.001 0.001"/>
@@ -369,5 +369,5 @@
 </joint>
 <joint name="joint2FrontRight" type="continuous">
-  <origin rpy="0 0 0" xyz="-0.041988 -0.0188 -0.072978"/>
+  <origin rpy="0.3 0 0" xyz="-0.041988 -0.0188 -0.072978"/>
   <parent link="link1FrontRight_1"/>
   <child link="link2FrontRight_1"/>
@@ -375,5 +375,5 @@
 </joint>
 <joint name="joint2BackLeft" type="continuous">
-  <origin rpy="0 0 0" xyz="0.041988 0.0188 -0.072978"/>
+  <origin rpy="0.8 0 0" xyz="0.041988 0.0188 -0.072978"/>
   <parent link="link1BackLeft_1"/>
   <child link="link2BackLeft_1"/>
@@ -381,5 +381,5 @@
 </joint>
 <joint name="joint2FrontLeft" type="continuous">
-  <origin rpy="0 0 0" xyz="0.042012 -0.0188 -0.072978"/>
+  <origin rpy="0.3 0 0" xyz="0.042012 -0.0188 -0.072978"/>
   <parent link="link1FrontLeft_1"/>
   <child link="link2FrontLeft_1"/>
@@ -387,5 +387,5 @@
 </joint>
 <joint name="joint2BackRight" type="continuous">
-  <origin rpy="0 0 0" xyz="-0.042012 0.0188 -0.072978"/>
+  <origin rpy="0.8 0 0" xyz="-0.042012 0.0188 -0.072978"/>
   <parent link="link1BackRight_1"/>
   <child link="link2BackRight_1"/>
@@ -393,17 +393,17 @@
 </joint>
 <joint name="joint3FrontRight" type="continuous">
-  <origin rpy="0 0 0" xyz="0.0 -1.2e-05 -0.256179"/>
+  <origin rpy="-0.1 0 0" xyz="0.0 0.221851 -0.1281"/>
   <parent link="link2FrontRight_1"/>
   <child link="link3FrontRight_1"/>
-  <axis xyz="-1.0 -0.0 -0.0"/>
+  <axis xyz="-1.0 0.0 0.0"/>
 </joint>
 <joint name="joint3BackLeft" type="continuous">
-  <origin rpy="0 0 0" xyz="-1e-06 1.2e-05 -0.256179"/>
+  <origin rpy="-0.2 0 0" xyz="-1e-06 -0.252284 -0.044498"/>
   <parent link="link2BackLeft_1"/>
   <child link="link3BackLeft__1"/>
-  <axis xyz="1.0 0.0 -0.0"/>
+  <axis xyz="1.0 -0.0 -0.0"/>
 </joint>
 <joint name="joint3FrontLeft" type="continuous">
-  <origin rpy="0 0 0" xyz="0.0 1.3e-05 -0.256179"/>
+  <origin rpy="-0.1 0 0" xyz="0.0 0.221863 -0.128079"/>
   <parent link="link2FrontLeft_1"/>
   <child link="link3FrontLeft_1"/>
@@ -411,17 +411,17 @@
 </joint>
 <joint name="joint3BackRight" type="continuous">
-  <origin rpy="0 0 0" xyz="-1e-06 -1.2e-05 -0.256179"/>
+  <origin rpy="-0.2 0 0" xyz="-1e-06 -0.252289 -0.044473"/>
   <parent link="link2BackRight_1"/>
   <child link="link3BackRight_1"/>
-  <axis xyz="-1.0 -0.0 -0.0"/>
+  <axis xyz="-1.0 0.0 -0.0"/>
 </joint>
 <joint name="joint4FrontRight" type="continuous">
-  <origin rpy="0 0 0" xyz="0.0 -1.3e-05 -0.284418"/>
+  <origin rpy="0 0 0" xyz="0.0 -0.18283 -0.217869"/>
   <parent link="link3FrontRight_1"/>
   <child link="link4FrontRight_1"/>
-  <axis xyz="-1.0 -0.0 -0.0"/>
+  <axis xyz="-1.0 0.0 0.0"/>
 </joint>
 <joint name="joint4BackLeft" type="continuous">
-  <origin rpy="0 0 0" xyz="0.0 1.3e-05 -0.284418"/>
+  <origin rpy="-0.7 0 0" xyz="0.0 0.18283 -0.217869"/>
   <parent link="link3BackLeft__1"/>
   <child link="link4BackLeft_1"/>
@@ -429,14 +429,14 @@
 </joint>
 <joint name="joint4FrontLeft" type="continuous">
-  <origin rpy="0 0 0" xyz="0.0 1.2e-05 -0.284418"/>
+  <origin rpy="0 0 0" xyz="0.0 -0.182811 -0.217885"/>
   <parent link="link3FrontLeft_1"/>
   <child link="link4FrontLeft_1"/>
-  <axis xyz="1.0 0.0 -0.0"/>
+  <axis xyz="1.0 -0.0 -0.0"/>
 </joint>
 <joint name="joint4BackRight" type="continuous">
-  <origin rpy="0 0 0" xyz="0.0 -1.3e-05 -0.284418"/>
+  <origin rpy="-0.7 0 0" xyz="1e-06 0.182811 -0.217885"/>
   <parent link="link3BackRight_1"/>
   <child link="link4FrontRight__1__1"/>
-  <axis xyz="-1.0 -0.0 -0.0"/>
+  <axis xyz="-1.0 0.0 -0.0"/>
 </joint>
 </robot>
