Commit message: New video exported for URDF

File: Matlab/urdf/quadruped_description/urdf/materials.xacro (robot description, xacro)
@@ -4,3 +4,9 @@
   <color rgba="0.700 0.700 0.700 1.000"/>
 </material>
+<material name="black_plastic">
+  <color rgba="0.300 0.300 0.300 1.000"/>
+</material>
+<material name="white_plastic">
+  <color rgba="1.000 1.000 1.000 1.000"/>
+</material>
 </robot>
